Commit message: quad

File: body.urdf (robot description, URDF)
Before this commit: robot robot, 3 links, 2 joints
Links:
- added link BackLowerLeg, mass 1; collision box size=0.2 0.2 1; visual box size=0.2 0.2 1
- added link FrontLowerLeg, mass 1; collision box size=0.2 0.2 1; visual box size=0.2 0.2 1
- added link LeftLeg, mass 1; collision box size=1 0.2 0.2; visual box size=1 0.2 0.2
- added link LeftLowerLeg, mass 1; collision box size=0.2 0.2 1; visual box size=0.2 0.2 1
- added link RightLeg, mass 1; collision box size=1 0.2 0.2; visual box size=1 0.2 0.2
- added link RightLowerLeg, mass 1; collision box size=0.2 0.2 1; visual box size=0.2 0.2 1
- link BackLeg: geometry collision box size=0.2 1 0.2; visual box size=0.2 1 0.2
- link FrontLeg: geometry collision box size=0.2 1 0.2; visual box size=0.2 1 0.2
Joints:
- added joint BackLeg_BackLowerLeg: type revolute, parent BackLeg, child BackLowerLeg, origin xyz=0 -1 0 rpy=0 0 0, axis 0 1 0, limit lower=-3.14159 upper=3.14159 effort=0.0 velocity=0.0
- added joint FrontLeg_FrontLowerLeg: type revolute, parent FrontLeg, child FrontLowerLeg, origin xyz=0 1 0 rpy=0 0 0, axis 0 1 0, limit lower=-3.14159 upper=3.14159 effort=0.0 velocity=0.0
- added joint LeftLeg_LeftLowerLeg: type revolute, parent LeftLeg, child LeftLowerLeg, origin xyz=-1 0 0 rpy=0 0 0, axis 0 1 0, limit lower=-3.14159 upper=3.14159 effort=0.0 velocity=0.0
- added joint RightLeg_RightLowerLeg: type revolute, parent RightLeg, child RightLowerLeg, origin xyz=1 0 0 rpy=0 0 0, axis 0 1 0, limit lower=-3.14159 upper=3.14159 effort=0.0 velocity=0.0
- added joint Torso_LeftLeg: type revolute, parent Torso, child LeftLeg, origin xyz=-0.5 0 1 rpy=0 0 0, axis 0 1 0, limit lower=-3.14159 upper=3.14159 effort=0.0 velocity=0.0
- added joint Torso_RightLeg: type revolute, parent Torso, child RightLeg, origin xyz=0.5 0 1 rpy=0 0 0, axis 0 1 0, limit lower=-3.14159 upper=3.14159 effort=0.0 velocity=0.0
- joint Torso_BackLeg: axis 0 1 0 -> 1 0 0; origin xyz=-0.5 0 1 rpy=0 0 0 -> xyz=0 -0.5 1 rpy=0 0 0
- joint Torso_FrontLeg: axis 0 1 0 -> 1 0 0; origin xyz=0.5 0 1 rpy=0 0 0 -> xyz=0 0.5 1 rpy=0 0 0

Commit message: asdf

File: body.urdf (robot description, URDF)
Before this commit: robot robot, 9 links, 8 joints
Links:
- link BackLeg: geometry collision box size=2 0.5 0.5; visual box size=2 0.5 0.5
- link BackLowerLeg: geometry collision box size=0.5 0.5 2; visual box size=0.5 0.5 2
- link FrontLeg: geometry collision box size=2 0.5 0.5; visual box size=2 0.5 0.5
- link FrontLowerLeg: geometry collision box size=0.5 0.5 2; visual box size=0.5 0.5 2
- link LeftLeg: geometry collision box size=2 0.5 0.5; visual box size=2 0.5 0.5
- link LeftLowerLeg: geometry collision box size=0.5 0.5 2; visual box size=0.5 0.5 2
- link RightLeg: geometry collision box size=2 0.5 0.5; visual box size=2 0.5 0.5
- link RightLowerLeg: geometry collision box size=0.5 0.5 2; visual box size=0.5 0.5 2
- link Torso: geometry collision box size=6 1 1; visual box size=6 1 1
Joints:
- joint BackLeg_BackLowerLeg: origin xyz=0 -1 0 rpy=0 0 0 -> xyz=-2.25 -0.25 0 rpy=0 0 0
- joint FrontLeg_FrontLowerLeg: origin xyz=0 1 0 rpy=0 0 0 -> xyz=-2.25 0.25 0 rpy=0 0 0
- joint LeftLeg_LeftLowerLeg: origin xyz=-1 0 0 rpy=0 0 0 -> xyz=-2.25 0.25 0 rpy=0 0 0
- joint RightLeg_RightLowerLeg: origin xyz=1 0 0 rpy=0 0 0 -> xyz=-2.25 -0.25 0 rpy=0 0 0
- joint Torso_BackLeg: axis 1 0 0 -> 0 1 0; origin xyz=0 -0.5 1 rpy=0 0 0 -> xyz=-2 -0.5 2 rpy=0 0 0
- joint Torso_FrontLeg: axis 1 0 0 -> 0 1 0; origin xyz=0 0.5 1 rpy=0 0 0 -> xyz=2 0.5 2 rpy=0 0 0
- joint Torso_LeftLeg: origin xyz=-0.5 0 1 rpy=0 0 0 -> xyz=-2 0.5 2 rpy=0 0 0
- joint Torso_RightLeg: origin xyz=0.5 0 1 rpy=0 0 0 -> xyz=2 -0.5 2 rpy=0 0 0

Commit message: commit!

File: body.urdf (robot description, URDF)
Before this commit: robot robot, 9 links, 8 joints
Links:
- removed link BackLeg
- removed link BackLowerLeg
- removed link FrontLeg
- removed link FrontLowerLeg
- removed link LeftLeg
- removed link LeftLowerLeg
- removed link RightLeg
- removed link RightLowerLeg
- removed link Torso
- added link 0, mass 1; collision box size=2.250747153246993 3.753565885202178 0.015951377131939726; visual box size=2.250747153246993 3.753565885202178 0.015951377131939726
- added link 1, mass 1; collision box size=2.57299783498819 3.0637457091502136 2.861636828081387; visual box size=2.57299783498819 3.0637457091502136 2.861636828081387
- added link 10, mass 1; collision box size=1.6955142940314443 2.8762511900454375 2.269419496305373; visual box size=1.6955142940314443 2.8762511900454375 2.269419496305373
- added link 2, mass 1; collision box size=3.5986848741267043 0.588055210826778 0.9968420715396364; visual box size=3.5986848741267043 0.588055210826778 0.9968420715396364
- added link 3, mass 1; collision box size=0.33409865908236425 0.5913192434299477 3.257127778935289; visual box size=0.33409865908236425 0.5913192434299477 3.257127778935289
- added link 4, mass 1; collision box size=3.1323497603515458 0.5333853559379218 0.428441497975097; visual box size=3.1323497603515458 0.5333853559379218 0.428441497975097
- added link 5, mass 1; collision box size=0.6135069508104696 1.7957009658385656 3.662322946159735; visual box size=0.6135069508104696 1.7957009658385656 3.662322946159735
- added link 6, mass 1; collision box size=3.5388313337452484 0.8780459043566209 3.1781155229194913; visual box size=3.5388313337452484 0.8780459043566209 3.1781155229194913
- added link 7, mass 1; collision box size=2.8326417337678116 2.9950087414309223 0.7428889189811136; visual box size=2.8326417337678116 2.9950087414309223 0.7428889189811136
- added link 8, mass 1; collision box size=3.1967274838801973 1.845540144723877 0.9485432934541023; visual box size=3.1967274838801973 1.845540144723877 0.9485432934541023
- added link 9, mass 1; collision box size=1.2849712325635316 2.6234110224803113 2.845042774445677; visual box size=1.2849712325635316 2.6234110224803113 2.845042774445677
Joints:
- removed joint BackLeg_BackLowerLeg
- removed joint FrontLeg_FrontLowerLeg
- removed joint LeftLeg_LeftLowerLeg
- removed joint RightLeg_RightLowerLeg
- removed joint Torso_BackLeg
- removed joint Torso_FrontLeg
- removed joint Torso_LeftLeg
- removed joint Torso_RightLeg
- added joint 0_1: type revolute, parent 0, child 1, origin xyz=0 1.876782942601089 3 rpy=0 0 0, axis 1 0 0, limit lower=-3.14159 upper=3.14159 effort=0.0 velocity=0.0
- added joint 1_2: type revolute, parent 1, child 2, origin xyz=0 3.0637457091502136 0 rpy=0 0 0, axis 0 0 1, limit lower=-3.14159 upper=3.14159 effort=0.0 velocity=0.0
- added joint 2_3: type revolute, parent 2, child 3, origin xyz=0 0.588055210826778 0 rpy=0 0 0, axis 1 0 0, limit lower=-3.14159 upper=3.14159 effort=0.0 velocity=0.0
- added joint 3_4: type revolute, parent 3, child 4, origin xyz=0 0.5913192434299477 0 rpy=0 0 0, axis 0 0 1, limit lower=-3.14159 upper=3.14159 effort=0.0 velocity=0.0
- added joint 4_5: type revolute, parent 4, child 5, origin xyz=0 0.5333853559379218 0 rpy=0 0 0, axis 1 0 0, limit lower=-3.14159 upper=3.14159 effort=0.0 velocity=0.0
- added joint 5_6: type revolute, parent 5, child 6, origin xyz=0 1.7957009658385656 0 rpy=0 0 0, axis 1 0 0, limit lower=-3.14159 upper=3.14159 effort=0.0 velocity=0.0
- added joint 6_7: type revolute, parent 6, child 7, origin xyz=0 0.8780459043566209 0 rpy=0 0 0, axis 0 1 0, limit lower=-3.14159 upper=3.14159 effort=0.0 velocity=0.0
- added joint 7_8: type revolute, parent 7, child 8, origin xyz=0 2.9950087414309223 0 rpy=0 0 0, axis 1 0 0, limit lower=-3.14159 upper=3.14159 effort=0.0 velocity=0.0
- added joint 8_9: type revolute, parent 8, child 9, origin xyz=0 1.845540144723877 0 rpy=0 0 0, axis 0 0 1, limit lower=-3.14159 upper=3.14159 effort=0.0 velocity=0.0
- added joint 9_10: type revolute, parent 9, child 10, origin xyz=0 2.6234110224803113 0 rpy=0 0 0, axis 1 0 0, limit lower=-3.14159 upper=3.14159 effort=0.0 velocity=0.0

Commit message: changes
cahnges

File: body.urdf (robot description, URDF)
Before this commit: robot robot, 11 links, 10 joints
Links:
- added link 11, mass 1; collision box size=0.5 1.0 4.0; visual box size=0.5 1.0 4.0
- added link 12, mass 1; collision box size=3.0 3.0 1.0; visual box size=3.0 3.0 1.0
- added link 13, mass 1; collision box size=3.5 1.5 1.5; visual box size=3.5 1.5 1.5
- link 0: geometry collision box size=4 1 1; visual box size=4 1 1
- link 1: geometry collision box size=3.5 3.5 5.0; visual box size=3.5 3.5 5.0
- link 10: geometry collision box size=0.5 4.0 5.0; visual box size=0.5 4.0 5.0
- link 2: geometry collision box size=1.0 2.0 4.5; visual box size=1.0 2.0 4.5
- link 3: geometry collision box size=2.5 3.0 0.5; visual box size=2.5 3.0 0.5
- link 4: geometry collision box size=0.5 0.5 2.0; visual box size=0.5 0.5 2.0
- link 5: geometry collision box size=2.0 1.5 5.0; visual box size=2.0 1.5 5.0
- link 6: geometry collision box size=2.5 1.0 3.5; visual box size=2.5 1.0 3.5
- link 7: geometry collision box size=2.5 3.5 2.0; visual box size=2.5 3.5 2.0
- link 8: geometry collision box size=3.5 0.5 5.0; visual box size=3.5 0.5 5.0
- link 9: geometry collision box size=2.5 3.5 3.0; visual box size=2.5 3.5 3.0
Joints:
- added joint 10_11: type revolute, parent 10, child 11, origin xyz=-0.5 2.0 -2.5 rpy=0 0 0, axis 0 0 1, limit lower=-3.14159 upper=3.14159 effort=0.0 velocity=0.0
- added joint 11_12: type revolute, parent 11, child 12, origin xyz=-0.5 0.5 -2.0 rpy=0 0 0, axis 0 0 1, limit lower=-3.14159 upper=3.14159 effort=0.0 velocity=0.0
- added joint 12_13: type revolute, parent 12, child 13, origin xyz=-3.0 1.5 -0.5 rpy=0 0 0, axis 0 1 0, limit lower=-3.14159 upper=3.14159 effort=0.0 velocity=0.0
- joint 0_1: origin xyz=0 1.876782942601089 3 rpy=0 0 0 -> xyz=-2 -0.5 10 rpy=0 0 0
- joint 1_2: origin xyz=0 3.0637457091502136 0 rpy=0 0 0 -> xyz=-3.5 -3.5 0 rpy=0 0 0
- joint 2_3: origin xyz=0 0.588055210826778 0 rpy=0 0 0 -> xyz=-1.0 -1.0 -2.25 rpy=0 0 0
- joint 3_4: origin xyz=0 0.5913192434299477 0 rpy=0 0 0 -> xyz=-2.5 0 -0.5 rpy=0 0 0
- joint 4_5: axis 1 0 0 -> 0 1 0; origin xyz=0 0.5333853559379218 0 rpy=0 0 0 -> xyz=-0.5 -0.25 -1.0 rpy=0 0 0
- joint 5_6: axis 1 0 0 -> 0 0 1; origin xyz=0 1.7957009658385656 0 rpy=0 0 0 -> xyz=-2.0 -0.75 -2.5 rpy=0 0 0
- joint 6_7: origin xyz=0 0.8780459043566209 0 rpy=0 0 0 -> xyz=-2.5 0 -3.5 rpy=0 0 0
- joint 7_8: axis 1 0 0 -> 0 0 1; origin xyz=0 2.9950087414309223 0 rpy=0 0 0 -> xyz=-2.5 -1.75 -1.0 rpy=0 0 0
- joint 8_9: axis 0 0 1 -> 1 0 0; origin xyz=0 1.845540144723877 0 rpy=0 0 0 -> xyz=-3.5 0 0 rpy=0 0 0
- joint 9_10: axis 1 0 0 -> 0 1 0; origin xyz=0 2.6234110224803113 0 rpy=0 0 0 -> xyz=-2.5 1.75 -1.5 rpy=0 0 0
